File: LED_shield/DMX.kicad_sch (KiCad schematic)
At the start: 14 parts, among them U401 SP3485EN, U402 SP3485EN

Commit message: Finish most of PCB design
Parts:
- renumbered C403 to C401, C404 to C402, C401 to C403, C402 to C404
Changed lines of the file:
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@@
 		(dnp no)
 		(fields_autoplaced yes)
-		(property "Reference" "#PWR0410"
+		(property "Reference" "#PWR0405"
 			(at 157.48 105.41 0)
 			(effects
@@
 			(project "LED_shield"
 				(path "/1ea5d53d-438b-4931-b69a-e3b85be65776/f6681d72-fe2e-40df-a5f5-abccfdd072e0"
-					(reference "#PWR0410")
+					(reference "#PWR0405")
 					(unit 1)
 				)
@@
 		(dnp no)
 		(fields_autoplaced yes)
-		(property "Reference" "#PWR0413"
+		(property "Reference" "#PWR0406"
 			(at 157.48 161.29 0)
 			(effects
@@
 			(project "LED_shield"
 				(path "/1ea5d53d-438b-4931-b69a-e3b85be65776/f6681d72-fe2e-40df-a5f5-abccfdd072e0"
-					(reference "#PWR0413")
+					(reference "#PWR0406")
 					(unit 1)
 				)
@@
 		(dnp no)
 		(fields_autoplaced yes)
-		(property "Reference" "#PWR0403"
+		(property "Reference" "#PWR0407"
 			(at 228.6 74.93 0)
 			(effects
@@
 			(project "LED_shield"
 				(path "/1ea5d53d-438b-4931-b69a-e3b85be65776/f6681d72-fe2e-40df-a5f5-abccfdd072e0"
-					(reference "#PWR0403")
+					(reference "#PWR0407")
 					(unit 1)
 				)
@@
 		(dnp no)
 		(fields_autoplaced yes)
-		(property "Reference" "#PWR0411"
+		(property "Reference" "#PWR0402"
 			(at 144.78 123.19 0)
 			(effects
@@
 			(project "LED_shield"
 				(path "/1ea5d53d-438b-4931-b69a-e3b85be65776/f6681d72-fe2e-40df-a5f5-abccfdd072e0"
-					(reference "#PWR0411")
+					(reference "#PWR0402")
 					(unit 1)
 				)
@@
 		(exclude_from_sim no)
 		(in_bom yes)
-		(on_board yes)
+		(on_board no)
 		(dnp no)
 		(fields_autoplaced yes)
@@
 		(exclude_from_sim no)
 		(in_bom yes)
-		(on_board yes)
+		(on_board no)
 		(dnp no)
 		(fields_autoplaced yes)
@@
 		(exclude_from_sim no)
 		(in_bom yes)
-		(on_board yes)
+		(on_board no)
 		(dnp no)
 		(fields_autoplaced yes)
@@
 		(exclude_from_sim no)
 		(in_bom yes)
-		(on_board yes)
-		(dnp no)
-		(fields_autoplaced yes)
-		(property "Reference" "C404"
+		(on_board no)
+		(dnp no)
+		(fields_autoplaced yes)
+		(property "Reference" "C402"
 			(at 147.701 109.2778 0)
 			(effects
@@
 			(project "LED_shield"
 				(path "/1ea5d53d-438b-4931-b69a-e3b85be65776/f6681d72-fe2e-40df-a5f5-abccfdd072e0"
-					(reference "C404")
+					(reference "C402")
 					(unit 1)
 				)
@@
 		(exclude_from_sim no)
 		(in_bom yes)
-		(on_board yes)
-		(dnp no)
-		(fields_autoplaced yes)
-		(property "Reference" "C403"
+		(on_board no)
+		(dnp no)
+		(fields_autoplaced yes)
+		(property "Reference" "C401"
 			(at 147.701 40.6978 0)
 			(effects
@@
 			(project ""
 				(path "/1ea5d53d-438b-4931-b69a-e3b85be65776/f6681d72-fe2e-40df-a5f5-abccfdd072e0"
-					(reference "C403")
+					(reference "C401")
 					(unit 1)
 				)
@@
 		(dnp no)
 		(fields_autoplaced yes)
-		(property "Reference" "#PWR0407"
+		(property "Reference" "#PWR0404"
 			(at 157.48 92.71 0)
 			(effects
@@
 			(project "LED_shield"
 				(path "/1ea5d53d-438b-4931-b69a-e3b85be65776/f6681d72-fe2e-40df-a5f5-abccfdd072e0"
-					(reference "#PWR0407")
+					(reference "#PWR0404")
 					(unit 1)
 				)
@@
 		(exclude_from_sim no)
 		(in_bom yes)
-		(on_board yes)
+		(on_board no)
 		(dnp no)
 		(fields_autoplaced yes)
@@
 		(dnp no)
 		(fields_autoplaced yes)
-		(property "Reference" "#PWR0402"
+		(property "Reference" "#PWR0409"
 			(at 241.3 36.83 0)
 			(effects
@@
 			(project ""
 				(path "/1ea5d53d-438b-4931-b69a-e3b85be65776/f6681d72-fe2e-40df-a5f5-abccfdd072e0"
-					(reference "#PWR0402")
+					(reference "#PWR0409")
 					(unit 1)
 				)
@@
 		(dnp no)
 		(fields_autoplaced yes)
-		(property "Reference" "#PWR0408"
+		(property "Reference" "#PWR0401"
 			(at 144.78 54.61 0)
 			(effects
@@
 			(project "LED_shield"
 				(path "/1ea5d53d-438b-4931-b69a-e3b85be65776/f6681d72-fe2e-40df-a5f5-abccfdd072e0"
-					(reference "#PWR0408")
+					(reference "#PWR0401")
 					(unit 1)
 				)
@@
 		(dnp no)
 		(fields_autoplaced yes)
-		(property "Reference" "#PWR0406"
+		(property "Reference" "#PWR0412"
 			(at 241.3 158.75 0)
 			(effects
@@
 			(project "LED_shield"
 				(path "/1ea5d53d-438b-4931-b69a-e3b85be65776/f6681d72-fe2e-40df-a5f5-abccfdd072e0"
-					(reference "#PWR0406")
+					(reference "#PWR0412")
 					(unit 1)
 				)
@@
 		(exclude_from_sim no)
 		(in_bom yes)
-		(on_board yes)
-		(dnp no)
-		(fields_autoplaced yes)
-		(property "Reference" "C401"
+		(on_board no)
+		(dnp no)
+		(fields_autoplaced yes)
+		(property "Reference" "C403"
 			(at 231.521 63.5578 0)
 			(effects
@@
 			(project ""
 				(path "/1ea5d53d-438b-4931-b69a-e3b85be65776/f6681d72-fe2e-40df-a5f5-abccfdd072e0"
-					(reference "C401")
+					(reference "C403")
 					(unit 1)
 				)
@@
 		(dnp no)
 		(fields_autoplaced yes)
-		(property "Reference" "#PWR0409"
+		(property "Reference" "#PWR0403"
 			(at 157.48 36.83 0)
 			(effects
@@
 			(project ""
 				(path "/1ea5d53d-438b-4931-b69a-e3b85be65776/f6681d72-fe2e-40df-a5f5-abccfdd072e0"
-					(reference "#PWR0409")
+					(reference "#PWR0403")
 					(unit 1)
 				)
@@
 		(dnp no)
 		(fields_autoplaced yes)
-		(property "Reference" "#PWR0405"
+		(property "Reference" "#PWR0408"
 			(at 228.6 143.51 0)
 			(effects
@@
 			(project "LED_shield"
 				(path "/1ea5d53d-438b-4931-b69a-e3b85be65776/f6681d72-fe2e-40df-a5f5-abccfdd072e0"
-					(reference "#PWR0405")
+					(reference "#PWR0408")
 					(unit 1)
 				)
@@
 		(exclude_from_sim no)
 		(in_bom yes)
-		(on_board yes)
+		(on_board no)
 		(dnp no)
 		(fields_autoplaced yes)
@@
 		(exclude_from_sim no)
 		(in_bom yes)
-		(on_board yes)
+		(on_board no)
 		(dnp no)
 		(fields_autoplaced yes)
@@
 		(exclude_from_sim no)
 		(in_bom yes)
-		(on_board yes)
+		(on_board no)
 		(dnp no)
 		(fields_autoplaced yes)
@@
 		(exclude_from_sim no)
 		(in_bom yes)
-		(on_board yes)
-		(dnp no)
-		(fields_autoplaced yes)
-		(property "Reference" "C402"
+		(on_board no)
+		(dnp no)
+		(fields_autoplaced yes)
+		(property "Reference" "C404"
 			(at 231.521 132.1378 0)
 			(effects
@@
 			(project "LED_shield"
 				(path "/1ea5d53d-438b-4931-b69a-e3b85be65776/f6681d72-fe2e-40df-a5f5-abccfdd072e0"
-					(reference "C402")
+					(reference "C404")
 					(unit 1)
 				)
@@
 		(exclude_from_sim no)
 		(in_bom yes)
-		(on_board yes)
+		(on_board no)
 		(dnp no)
 		(fields_autoplaced yes)
@@
 		(dnp no)
 		(fields_autoplaced yes)
-		(property "Reference" "#PWR0404"
+		(property "Reference" "#PWR0411"
 			(at 241.3 105.41 0)
 			(effects
@@
 			(project "LED_shield"
 				(path "/1ea5d53d-438b-4931-b69a-e3b85be65776/f6681d72-fe2e-40df-a5f5-abccfdd072e0"
-					(reference "#PWR0404")
+					(reference "#PWR0411")
 					(unit 1)
 				)
@@
 		(dnp no)
 		(fields_autoplaced yes)
-		(property "Reference" "#PWR0401"
+		(property "Reference" "#PWR0410"
 			(at 241.3 90.17 0)
 			(effects
@@
 			(project ""
 				(path "/1ea5d53d-438b-4931-b69a-e3b85be65776/f6681d72-fe2e-40df-a5f5-abccfdd072e0"
-					(reference "#PWR0401")
+					(reference "#PWR0410")
 					(unit 1)
 				)
@@
 		(exclude_from_sim no)
 		(in_bom yes)
-		(on_board yes)
+		(on_board no)
 		(dnp no)
 		(fields_autoplaced yes)
@@
 		(exclude_from_sim no)
 		(in_bom yes)
-		(on_board yes)
-		(dnp no)
-		(fields_autoplaced yes)
+		(on_board no)
+		(dnp no)
+		(fields_autoplaced yes)
